Commit message: aight dees zou moeten werken

File: src/isfr_bot_description/urdf/IsfrFullRobot.urdf (robot description, URDF)
Before this commit: robot IsfrFullRobot, 22 links, 21 joints
Links:
- removed link base_footprint
- removed link camera_depth_frame
- removed link camera_depth_optical_frame
- removed link camera_link
- removed link camera_rgb_frame
- removed link camera_rgb_optical_frame
- removed link caster_back_left_link
- removed link caster_back_right_link
- removed link end_effector_link
- removed link gripper_left_link
- removed link gripper_right_link
- removed link link1
- removed link link2
- removed link link3
- removed link link4
- removed link link5
- removed link world
- link base_link: mass 1.3729096e+00 -> None; geometry 
- link base_scan: mass 0.114 -> None; geometry 
- link wheel_left_link: mass 2.8498940e-02 -> None; geometry 
- link wheel_right_link: mass 2.8498940e-02 -> None; geometry 
Joints:
- removed joint arm_base_joint
- removed joint base_joint
- removed joint camera_depth_joint
- removed joint camera_depth_optical_joint
- removed joint camera_joint
- removed joint camera_rgb_joint
- removed joint camera_rgb_optical_joint
- removed joint caster_back_left_joint
- removed joint caster_back_right_joint
- removed joint end_effector_joint
- removed joint gripper_left_joint
- removed joint gripper_right_joint
- removed joint joint1
- removed joint joint2
- removed joint joint3
- removed joint joint4
- removed joint scan_joint
- removed joint wheel_left_joint
- removed joint wheel_right_joint
- removed joint world_fixed
- added joint left_wheel_joint: type continuous, parent base_link, child wheel_left_link, origin xyz=0 0.144 0.023 rpy=0 0 0, axis 0 1 0
- added joint lidar_joint: type fixed, parent base_link, child base_scan, origin xyz=-0.064 0 0.1015 rpy=0 0 0
- added joint right_wheel_joint: type continuous, parent base_link, child wheel_right_link, origin xyz=0 -0.144 0.023 rpy=0 0 0, axis 0 1 0
- joint imu_joint: origin xyz=0.0 0 0.068 rpy=0 0 0 -> xyz=-0.064 0 0.1015 rpy=0 0 0

Commit message: nu kan deze repo normaal gezien evenveel als de andere (+ ook lidar die hier wel werkt)

File: src/isfr_bot_description/urdf/IsfrFullRobot.urdf (robot description, URDF)
Before this commit: robot isfr_bot, 5 links, 4 joints
Links:
- removed link base_link
- removed link base_scan
- removed link imu_link
- removed link wheel_left_link
- removed link wheel_right_link
Joints:
- removed joint imu_joint
- removed joint left_wheel_joint
- removed joint lidar_joint
- removed joint right_wheel_joint
